Commit message: unbreaking gazebo

File: description/gazebo_control.xacro (robot description, xacro)
@@ -6,6 +6,6 @@
                 <left_joint>left_wheel_joint</left_joint>
                 <right_joint>right_wheel_joint</right_joint>
-                <wheel_separation>0.35</wheel_separation>
-                <wheel_diameter>0.1</wheel_diameter>
+                <wheel_separation>0.2</wheel_separation>
+                <wheel_diameter>0.065</wheel_diameter>
                 <!-- Limits -->
                 <max_wheel_torque>200</max_wheel_torque>

File: description/robot.urdf.xacro (robot description, xacro)
@@ -1,6 +1,13 @@
 <?xml version="1.0"?>
 <robot xmlns:xacro="http://www.ros.org/wiki/xacro"  name="robot">
-    <xacro:include filename="robot_core.xacro" />
-    <xacro:include filename="ros2_control.xacro"/>
+    <xacro:arg name="use_ros2_control" default="true"/>
+    <xacro:arg name="sim_mode" default="false"/>
+    <xacro:include filename="robot_core.xacro"/>
+    <xacro:if value="$(arg use_ros2_control)">
+        <xacro:include filename="ros2_control.xacro" />
+    </xacro:if>
+    <xacro:unless value="$(arg use_ros2_control)">
+        <xacro:include filename="gazebo_control.xacro" />
+    </xacro:unless>
     <xacro:include filename="lidar.xacro" />
     <!-- <xacro:include filename="gazebo_control.xacro"/> -->

File: description/robot_core.xacro (robot description, xacro)
@@ -12,5 +12,5 @@
     <xacro:property name="wheel_offset_y" value="${chassis_width/2}"/>
     <xacro:property name="wheel_offset_z" value="${wheel_radius/2}"/>
-    <xacro:property name="caster_wheel_radius" value="0.015"/>
+    <xacro:property name="caster_wheel_radius" value="0.010"/>
     <xacro:property name="caster_wheel_mass" value="0.01"/>
     <xacro:property name="caster_wheel_offset_x" value="0.02"/>

File: description/ros2_control.xacro (robot description, xacro)
@@ -1,33 +1,36 @@
 <?xml version="1.0"?>
 <robot xmlns:xacro="http://www.ros.org/wiki/xacro">
-    <ros2_control name="RealRobot" type="system">
-            <hardware>
-                <plugin>diffdrive_arduino/DiffDriveArduino</plugin>
-                <param name="left_wheel_name">left_wheel_joint</param>
-                <param name="right_wheel_name">right_wheel_joint</param>
-                <param name="loop_rate">30</param>
-                <param name="device">/dev/ttyACM0</param>
-                <param name="baud_rate">57600</param>
-                <param name="timeout">1000</param>
-                <param name="enc_counts_per_rev">1550</param>
-            </hardware>s
-            <joint name="left_wheel_joint">
-                <command_interface name="velocity">
-                    <param name="min">-10</param>
-                    <param name="max">10</param>
-                </command_interface>
-                <state_interface name="position" />
-                <state_interface name="velocity" />
-            </joint>
-            <joint name="right_wheel_joint">
-                <command_interface name="velocity">s
-                    <param name="min">-10</param>
-                    <param name="max">10</param>
-                </command_interface>
-                <state_interface name="velocity" />
-                <state_interface name="position" />
-            </joint>
-    </ros2_control>
-        <!-- <ros2_control name="GazeboSystem" type="system">
+    <xacro:unless value="$(arg sim_mode)">
+        <ros2_control name="RealRobot" type="system">
+                <hardware>
+                    <plugin>diffdrive_arduino/DiffDriveArduino</plugin>
+                    <param name="left_wheel_name">left_wheel_joint</param>
+                    <param name="right_wheel_name">right_wheel_joint</param>
+                    <param name="loop_rate">30</param>
+                    <param name="device">/dev/ttyACM0</param>
+                    <param name="baud_rate">57600</param>
+                    <param name="timeout">1000</param>
+                    <param name="enc_counts_per_rev">1550</param>
+                </hardware>s
+                <joint name="left_wheel_joint">
+                    <command_interface name="velocity">
+                        <param name="min">-10</param>
+                        <param name="max">10</param>
+                    </command_interface>
+                    <state_interface name="position" />
+                    <state_interface name="velocity" />
+                </joint>
+                <joint name="right_wheel_joint">
+                    <command_interface name="velocity">s
+                        <param name="min">-10</param>
+                        <param name="max">10</param>
+                    </command_interface>
+                    <state_interface name="velocity" />
+                    <state_interface name="position" />
+                </joint>
+        </ros2_control>
+    </xacro:unless>
+    <xacro:if value="$(arg sim_mode)">
+        <ros2_control name="GazeboSystem" type="system">
             <hardware>
                 <plugin>gazebo_ros2_control/GazeboSystem</plugin>
@@ -49,8 +52,10 @@
                 <state_interface name="position" />
             </joint>
-    </ros2_control> -->
+        </ros2_control>
+    </xacro:if>
     <gazebo>
         <plugin  name="gazebo_ros2_control" filename="libgazebo_ros2_control.so">
             <parameters>$(find my_bot)/config/my_controllers.yaml</parameters>
+            <parameters>$(find my_bot)/config/gaz_ros2_ctl_use_sim.yaml</parameters>
         </plugin>
     </gazebo>
